Commit message: urdf joints

File: robotmodel.urdf (robot description, URDF)
Before this commit: robot tank1, 1 links, 0 joints
Links:
- added link lwheel; visual cylinder length=0.005 radius=0.026
- added link rwheel; visual cylinder length=0.005 radius=0.026
Joints:
- added joint base_to_lwheel: type continuous, parent base_link, child lwheel, origin xyz=0 0.08 0.026 rpy=1.5708 0 0
- added joint base_to_rwheel: type continuous, parent base_link, child rwheel, origin xyz=0 -0.08 0.026 rpy=-1.5708 0 0

Commit message: urdf

File: robotmodel.urdf (robot description, URDF)
Before this commit: robot mbot, 3 links, 2 joints
Links:
- added link imu
- added link laser; visual cylinder length=0.01 radius=0.03
- link lwheel: geometry visual cylinder length=0.005 radius=0.016
- link rwheel: geometry visual cylinder length=0.005 radius=0.016
Joints:
- added joint joint_base_imu: type fixed, parent base_link, child imu, origin xyz=0.0 0.0 0.0 rpy=3.141592 0 0
- added joint joint_sensor_laser: type fixed, parent base_link, child laser, origin xyz=0.0202 -0.02 0.10 rpy=0 0 3.08
- joint base_to_lwheel: origin xyz=0 0.08 0.026 rpy=1.5708 0 0 -> xyz=0 0.08 0.016 rpy=0 0 1.5708
- joint base_to_rwheel: origin xyz=0 -0.08 0.026 rpy=-1.5708 0 0 -> xyz=0 -0.08 0.016 rpy=0 0 -1.5708

Commit message: CAD model for the caster wheel robot

File: robotmodel.urdf (robot description, URDF)
Before this commit: robot mbot, 5 links, 4 joints
Links:
- link base_link: geometry visual mesh filename=package://system_setup/CAD/3wheels.stl

Commit message: urdf updated

File: robotmodel.urdf (robot description, URDF)
Before this commit: robot mbot, 5 links, 4 joints
Joints:
- joint joint_base_imu: origin xyz=0.0 0.0 0.0 rpy=3.141592 0 0 -> xyz=0.0 0.0 0.0 rpy=3.14159265359 0 0
- joint joint_sensor_laser: origin xyz=0.0202 -0.02 0.10 rpy=0 0 3.08 -> xyz=-0.0733551 -0.0160634 0.16 rpy=0 0 -0.0336378
